File: PCB_kicad/alpha_pro_micro.kicad_pcb (KiCad board)
At the start: 2 copper layers, 192.9 x 59.5 mm, 64 parts, among them J1 Conn_01x03, K1 KEYSW, K10 KEYSW, K11 KEYSW, K12 KEYSW, K13 KEYSW, K14 KEYSW, K15 KEYSW, K16 KEYSW, K17 KEYSW, K18 KEYSW, K19 KEYSW, K2 KEYSW, K20 KEYSW, K21 KEYSW, K22 KEYSW, K23 KEYSW, K24 KEYSW, K25 KEYSW, K26 KEYSW, K27 KEYSW, K28 KEYSW, K3 KEYSW, K4 KEYSW, K5 KEYSW, K6 KEYSW, K7 KEYSW, K8 KEYSW, K9 KEYSW, SW1 SW_Push, U1 ProMicro

Commit message: v2.2
Other:
- board text added: "v2.2"
- board text removed: "v2.0"
- board text removed: "v2.1"
Changed lines of the file:
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@@
     (34 B.Paste user)
     (35 F.Paste user)
-    (36 B.SilkS user hide)
-    (37 F.SilkS user hide)
+    (36 B.SilkS user)
+    (37 F.SilkS user)
     (38 B.Mask user)
     (39 F.Mask user hide)
@@
     (effects (font (size 0.6 0.6) (thickness 0.15)))
   )
-  (gr_text v2.0 (at 83.391137 154.393424) (layer B.SilkS)
+  (gr_text v2.2 (at 83.391137 154.393424) (layer B.SilkS)
     (effects (font (size 1.5 1.5) (thickness 0.3) italic) (justify mirror))
   )
-  (gr_text v2.1 (at 243.179997 156.102844) (layer F.SilkS)
+  (gr_text v2.2 (at 243.179997 156.102844) (layer F.SilkS)
     (effects (font (size 1.5 1.5) (thickness 0.3) italic))
   )
@@
   (segment (start 72.628125 126.285625) (end 72.628125 134.471172) (width 0.25) (layer F.Cu) (net 32) (status 10))
   (segment (start 76.2 103.6375) (end 74.3 105.5375) (width 0.25) (layer F.Cu) (net 32) (status 30))
-  (segment (start 76.2 122.6875) (end 77.666992 121.220508) (width 0.25) (layer B.Cu) (net 32) (status 10))
-  (segment (start 106.059883 121.220508) (end 106.68 121.840625) (width 0.25) (layer B.Cu) (net 32) (status 20))
-  (segment (start 81.632227 121.220508) (end 83.715819 123.3041) (width 0.25) (layer B.Cu) (net 32))
-  (segment (start 77.666992 121.220508) (end 81.632227 121.220508) (width 0.25) (layer B.Cu) (net 32))
-  (segment (start 83.715819 123.3041) (end 87.808595 123.3041) (width 0.25) (layer B.Cu) (net 32))
-  (segment (start 87.808595 123.3041) (end 89.892187 121.220508) (width 0.25) (layer B.Cu) (net 32))
-  (segment (start 89.892187 121.220508) (end 106.059883 121.220508) (width 0.25) (layer B.Cu) (net 32))
   (segment (start 76.2 122.6875) (end 74.3 124.5875) (width 0.25) (layer B.Cu) (net 32) (status 30))
   (segment (start 85.725 141.7375) (end 83.825 143.6375) (width 0.25) (layer F.Cu) (net 32) (status 30))
+  (segment (start 105.739375 120.9) (end 106.68 121.840625) (width 0.25) (layer B.Cu) (net 32))
+  (segment (start 76.2 122.6875) (end 77.666992 121.220508) (width 0.25) (layer B.Cu) (net 32))
+  (segment (start 81.632227 121.220508) (end 83.715819 123.3041) (width 0.25) (layer B.Cu) (net 32))
+  (segment (start 83.715819 123.3041) (end 87.808595 123.3041) (width 0.25) (layer B.Cu) (net 32))
+  (segment (start 77.666992 121.220508) (end 81.632227 121.220508) (width 0.25) (layer B.Cu) (net 32))
+  (segment (start 87.808595 123.3041) (end 90.212695 120.9) (width 0.25) (layer B.Cu) (net 32))
+  (segment (start 90.212695 120.9) (end 105.739375 120.9) (width 0.25) (layer B.Cu) (net 32))
   (segment (start 91.44 126.0475) (end 91.44 135.641953) (width 0.25) (layer F.Cu) (net 33) (status 10))
   (segment (start 91.44 135.641953) (end 100.965 145.166953) (width 0.25) (layer F.Cu) (net 33) (status 20))
